Commit message: wrote cpp code for generating a casadi function for forward dynamics

File: models/flexible_arm_jiminy.urdf (robot description, URDF)
Before this commit: robot flexible_arm, 7 links, 6 joints
Joints:
- joint base_to_link1: limit lower=-3.14159 upper=3.14159 effort=100.0 velocity=3.14 -> lower=0.0 upper=1.0 effort=100.0 velocity=0.5
- joint link1_to_link2: limit lower=-3.14159 upper=3.14159 effort=100.0 velocity=3.14 -> lower=0.0 upper=1.0 effort=100.0 velocity=0.5; type revolute -> fixed
- joint link2_to_link3: limit lower=-3.14159 upper=3.14159 effort=100.0 velocity=3.14 -> lower=0.0 upper=1.0 effort=100.0 velocity=0.5; type revolute -> fixed
- joint link3_to_link4: limit lower=-3.14159 upper=3.14159 effort=100.0 velocity=3.14 -> lower=0.0 upper=1.0 effort=100.0 velocity=0.5; type revolute -> fixed
- joint link4_to_link5: limit lower=-3.14159 upper=3.14159 effort=100.0 velocity=3.14 -> lower=0.0 upper=1.0 effort=100.0 velocity=0.5; type revolute -> fixed

Commit message: Comparing jiminy simulation trajectories with mine

File: models/flexible_arm_jiminy.urdf (robot description, URDF)
Before this commit: robot flexible_arm, 7 links, 6 joints
Links:
- removed link load
Joints:
- removed joint link5_to_load
- joint base_to_link1: limit lower=0.0 upper=1.0 effort=100.0 velocity=0.5 -> lower=-3.14159 upper=3.14159 effort=100.0 velocity=3.14; origin xyz=0 0 0 rpy=1.57 0 0 -> xyz=0 0 0 rpy=1.57079632679489661923 0 0
- joint link1_to_link2: limit lower=0.0 upper=1.0 effort=100.0 velocity=0.5 -> lower=-3.14159 upper=3.14159 effort=100.0 velocity=3.14
- joint link2_to_link3: limit lower=0.0 upper=1.0 effort=100.0 velocity=0.5 -> lower=-3.14159 upper=3.14159 effort=100.0 velocity=3.14
- joint link3_to_link4: limit lower=0.0 upper=1.0 effort=100.0 velocity=0.5 -> lower=-3.14159 upper=3.14159 effort=100.0 velocity=3.14
- joint link4_to_link5: limit lower=0.0 upper=1.0 effort=100.0 velocity=0.5 -> lower=-3.14159 upper=3.14159 effort=100.0 velocity=3.14

File: models/flexible_arm_v1.urdf (robot description, URDF)
Before this commit: robot flexible_arm, 7 links, 6 joints
Links:
- removed link load
Joints:
- removed joint link5_to_load
- joint base_to_link1: origin xyz=0 0 0 rpy=1.57 0 0 -> xyz=0 0 0 rpy=1.57079632679489661923 0 0
