Commit message: implemented a code for obtaining lumped model (rigid finite element) parameters for a beam. Modified the three segment urdf according to calculated parameters

File: models/three_segments/flexible_arm_1dof_3s.urdf (robot description, URDF)
Before this commit: robot flexible_arm, 5 links, 4 joints
Links:
- added link virtual_link4, mass 0.06558333333333334; visual box size=0.08333333333333333 0.025 0.01
- link virtual_link1: mass 1.333333333 -> 0.06558333333333334; geometry visual box size=0.08333333333333333 0.025 0.01
- link virtual_link2: mass 1.333333333 -> 0.13116666666666668
- link virtual_link3: mass 1.333333333 -> 0.13116666666666668
Joints:
- removed joint virtual_link3_to_load
- added joint passive_joint3: type revolute, parent virtual_link3, child virtual_link4, origin xyz=0.166666667 0 0 rpy=0 0 0, axis 0 0 1, limit lower=-3.14159 upper=3.14159 effort=100.0 velocity=3.14
- added joint virtual_link4_to_load: type fixed, parent virtual_link4, child load, origin xyz=0.08333333333333333 0 0 rpy=0 0 0, axis 0 0 1
- joint passive_joint1: origin xyz=0.166666667 0 0 rpy=0 0 0 -> xyz=0.08333333333333333 0 0 rpy=0 0 0
