Commit message: forget to add files :(

File: models/five_segments/flexible_arm_1dof_5s.urdf (robot description, URDF)
Before this commit: robot flexible_arm, 7 links, 6 joints
Links:
- removed link link1
- removed link link2
- removed link link3
- removed link link4
- removed link link5
- added link virtual_link1, mass 0.8; visual box size=0.1 0.025 0.01
- added link virtual_link2, mass 0.8; visual box size=0.1 0.025 0.01
- added link virtual_link3, mass 0.8; visual box size=0.1 0.025 0.01
- added link virtual_link4, mass 0.8; visual box size=0.1 0.025 0.01
- added link virtual_link5, mass 0.8; visual box size=0.1 0.025 0.01
Joints:
- removed joint base_to_link1
- removed joint link1_to_link2
- removed joint link2_to_link3
- removed joint link3_to_link4
- removed joint link4_to_link5
- removed joint link5_to_load
- added joint active_joint: type revolute, parent world, child virtual_link1, origin xyz=0 0 0 rpy=1.57 0 0, axis 0 0 1, limit lower=-3.14159 upper=3.14159 effort=100.0 velocity=3.14
- added joint passive_joint1: type revolute, parent virtual_link1, child virtual_link2, origin xyz=0.1 0 0 rpy=0 0 0, axis 0 0 1, limit lower=-3.14159 upper=3.14159 effort=100.0 velocity=3.14
- added joint passive_joint2: type revolute, parent virtual_link2, child virtual_link3, origin xyz=0.1 0 0 rpy=0 0 0, axis 0 0 1, limit lower=-3.14159 upper=3.14159 effort=100.0 velocity=3.14
- added joint passive_joint3: type revolute, parent virtual_link3, child virtual_link4, origin xyz=0.1 0 0 rpy=0 0 0, axis 0 0 1, limit lower=-3.14159 upper=3.14159 effort=100.0 velocity=3.14
- added joint passive_joint4: type revolute, parent virtual_link4, child virtual_link5, origin xyz=0.1 0 0 rpy=0 0 0, axis 0 0 1, limit lower=-3.14159 upper=3.14159 effort=100.0 velocity=3.14
- added joint virtual_link5_to_load: type fixed, parent virtual_link5, child load, origin xyz=0.1 0 0 rpy=0 0 0, axis 0 0 1

Commit message: Modified models so that they correspond to an actual beam parameters. It is correcyt now for 3, 5 and 10 segment models

File: models/five_segments/flexible_arm_1dof_5s.urdf (robot description, URDF)
Before this commit: robot flexible_arm, 7 links, 6 joints
Links:
- added link virtual_link6, mass 0.03935; visual box size=0.05 0.025 0.01
- link virtual_link1: mass 0.8 -> 0.03935; geometry visual box size=0.05 0.025 0.01
- link virtual_link2: mass 0.8 -> 0.0787
- link virtual_link3: mass 0.8 -> 0.0787
- link virtual_link4: mass 0.8 -> 0.0787
- link virtual_link5: mass 0.8 -> 0.0787
Joints:
- removed joint virtual_link5_to_load
- added joint passive_joint5: type revolute, parent virtual_link5, child virtual_link6, origin xyz=0.1 0 0 rpy=0 0 0, axis 0 0 1, limit lower=-3.14159 upper=3.14159 effort=100.0 velocity=3.14
- added joint virtual_link6_to_load: type fixed, parent virtual_link6, child load, origin xyz=0.05 0 0 rpy=0 0 0, axis 0 0 1
- joint passive_joint1: origin xyz=0.1 0 0 rpy=0 0 0 -> xyz=0.05 0 0 rpy=0 0 0

File: models/ten_segments/flexible_arm_1dof_10s.urdf (robot description, URDF)
Before this commit: robot flexible_arm, 12 links, 11 joints
Links:
- added link virtual_link11, mass 0.019675; visual box size=0.025 0.025 0.01
- link virtual_link1: mass 0.4 -> 0.019675; geometry visual box size=0.025 0.025 0.01
- link virtual_link10: mass 0.4 -> 0.03935
- link virtual_link2: mass 0.4 -> 0.03935
- link virtual_link3: mass 0.4 -> 0.03935
- link virtual_link4: mass 0.4 -> 0.03935
- link virtual_link5: mass 0.4 -> 0.03935
- link virtual_link6: mass 0.4 -> 0.03935
- link virtual_link7: mass 0.4 -> 0.03935
- link virtual_link8: mass 0.4 -> 0.03935
- link virtual_link9: mass 0.4 -> 0.03935
Joints:
- removed joint virtual_link10_to_load
- added joint passive_joint10: type revolute, parent virtual_link10, child virtual_link11, origin xyz=0.05 0 0 rpy=0 0 0, axis 0 0 1, limit lower=-3.14159 upper=3.14159 effort=100.0 velocity=3.14
- added joint virtual_link11_to_load: type fixed, parent virtual_link11, child load, origin xyz=0.025 0 0 rpy=0 0 0, axis 0 0 1
- joint passive_joint1: origin xyz=0.05 0 0 rpy=0 0 0 -> xyz=0.025 0 0 rpy=0 0 0
