Commit message: Created URDF for a 3 dof robot with 2 flexible links and rigid base link. Generated kinematics and dynamics funtions for the model. Created a symbolic model to be used in MPC. Tested the model.

File: models/one_dof/ten_segments/flexible_arm_1dof_10s.urdf (robot description, URDF)
Before this commit: robot flexible_arm, 13 links, 12 joints
Joints:
- removed joint virtual_link11_to_load
- added joint last_link_to_load: type fixed, parent virtual_link11, child load, origin xyz=0.025 0 0 rpy=0 0 0, axis 0 0 1
