Commit message: fixed small error in defning the end-effector frame

File: models/one_dof/five_segments/flexible_arm_1dof_5s.urdf (robot description, URDF)
Before this commit: robot flexible_arm, 8 links, 7 joints
Joints:
- removed joint virtual_link6_to_load
- added joint last_link_to_load: type fixed, parent virtual_link6, child load, origin xyz=0.05 0 0 rpy=0 0 0, axis 0 0 1

File: models/one_dof/three_segments/flexible_arm_1dof_3s.urdf (robot description, URDF)
Before this commit: robot flexible_arm, 6 links, 5 joints
Joints:
- removed joint virtual_link4_to_load
- added joint last_link_to_load: type fixed, parent virtual_link4, child load, origin xyz=0.08333333333333333 0 0 rpy=0 0 0, axis 0 0 1
