Commit message: small modification for visualization

File: flexible_arm_ws/src/fa_setup/urdf/fa_setup_descr.xacro (robot description, xacro)
@@ -14,8 +14,8 @@
 </xacro:macro>
 <!-- Wall parameters -->
-<xacro:property name="d_origin_to_wall" value="0.5" />
+<xacro:property name="d_origin_to_wall" value="0.04" />
 <xacro:property name="wall_thickness" value="0.075" />
 <xacro:property name="wall_height" value="1.0" />
-<xacro:property name="wall_width" value="1.5" />
+<xacro:property name="wall_width" value="2" />
 <!-- Flexible arm -->
 <!-- <xacro:include filename="$(find fa_setup)/urdf/flexible_arm_3dof_0s.urdf" /> -->
@@ -24,5 +24,5 @@
 <link name = "wall_link">
     <visual>
-        <origin xyz="${d_origin_to_wall} 0 ${wall_height/2}" rpy="0 0 0" />
+        <origin xyz="${d_origin_to_wall} ${wall_thickness/2} ${wall_height/2}" rpy="0 0 0" />
         <geometry>
             <box size="${wall_width} ${wall_thickness} ${wall_height}"/>
@@ -40,5 +40,5 @@
     <parent link = "world" />
     <child link = "wall_link" />
-    <origin xyz = "${d_origin_to_wall} 0 0" />
+    <origin xyz = "0 ${d_origin_to_wall} 0" />
 </joint>
 </robot>
