Commit message: Added catkin workspace for visualizing the robot in Rviz and generating figures. In the worksapce there is a xacro file that takes 10 segment robots urdf and adds a wall into the environment. Additionally added files for generating figures for the beneluz conference etc

File: models/three_dof/ten_segments/flexible_arm_3dof_10s.urdf (robot description, URDF)
Before this commit: robot flexible_arm, 25 links, 24 joints
Links:
- link load: geometry visual sphere radius=0.0005

Commit message: Added wall to 10 segment discretiszation of the flexible robot

File: models/three_dof/ten_segments/flexible_arm_3dof_10s.urdf (robot description, URDF)
Before this commit: robot flexible_arm, 25 links, 24 joints
Links:
- added link wall_link, mass 15; collision box size=0.075 2 1; visual box size=2 0.075 1
Joints:
- added joint world_to_wall: type fixed, parent world, child wall_link, origin xyz=0 -0.15 0
