Commit message: Found and corrected some errors/bugs in the link parameter estimation and stiffness estimation. Added 1 segment model. The comparison between different approximations is improved: now all the models get the same input

File: models/three_dof/five_segments/flexible_arm_3dof_5s.urdf (robot description, URDF)
Before this commit: robot flexible_arm, 15 links, 14 joints
Links:
- link virtual_link2_1: geometry visual box size=0.05 0.002 0.05
- link virtual_link2_2: geometry visual box size=0.1 0.002 0.05
- link virtual_link2_3: geometry visual box size=0.1 0.002 0.05
- link virtual_link2_4: geometry visual box size=0.1 0.002 0.05
- link virtual_link2_5: geometry visual box size=0.1 0.002 0.05
- link virtual_link2_6: geometry visual box size=0.05 0.002 0.05
- link virtual_link3_1: geometry visual box size=0.05 0.002 0.05
- link virtual_link3_2: geometry visual box size=0.1 0.002 0.05
- link virtual_link3_3: geometry visual box size=0.1 0.002 0.05
- link virtual_link3_4: geometry visual box size=0.1 0.002 0.05
- link virtual_link3_5: geometry visual box size=0.1 0.002 0.05
- link virtual_link3_6: geometry visual box size=0.05 0.002 0.05

File: models/three_dof/one_segments/flexible_arm_3dof_1s.urdf (robot description, URDF)
Before this commit: robot flexible_arm, 9 links, 8 joints
Links:
- removed link virtual_link2_3
- removed link virtual_link3_3
- link virtual_link2_1: mass 0.098375 -> 0.19675; geometry visual box size=0.25 0.002 0.05
- link virtual_link3_1: mass 0.098375 -> 0.19675; geometry visual box size=0.25 0.002 0.05
Joints:
- removed joint passive_joint2
- removed joint passive_joint3_2
- joint active_joint3: origin xyz=0.125 0 0 rpy=0 0 0 -> xyz=0.25 0 0 rpy=0 0 0; parent virtual_link2_3 -> virtual_link2_2
- joint last_link_to_load: origin xyz=0.125 0 0 rpy=0 0 0 -> xyz=0.25 0 0 rpy=0 0 0; parent virtual_link3_3 -> virtual_link3_2
- joint passive_joint1: origin xyz=0.125 0 0 rpy=0 0 0 -> xyz=0.25 0 0 rpy=0 0 0
- joint passive_joint3_1: origin xyz=0.125 0 0 rpy=0 0 0 -> xyz=0.25 0 0 rpy=0 0 0

File: models/three_dof/ten_segments/flexible_arm_3dof_10s.urdf (robot description, URDF)
Before this commit: robot flexible_arm, 25 links, 24 joints
Links:
- link virtual_link2_1: geometry visual box size=0.025 0.002 0.05
- link virtual_link2_10: geometry visual box size=0.05 0.002 0.05
- link virtual_link2_11: geometry visual box size=0.025 0.002 0.05
- link virtual_link2_2: geometry visual box size=0.05 0.002 0.05
- link virtual_link2_3: geometry visual box size=0.05 0.002 0.05
- link virtual_link2_4: geometry visual box size=0.05 0.002 0.05
- link virtual_link2_5: geometry visual box size=0.05 0.002 0.05
- link virtual_link2_6: geometry visual box size=0.05 0.002 0.05
- link virtual_link2_7: geometry visual box size=0.05 0.002 0.05
- link virtual_link2_8: geometry visual box size=0.05 0.002 0.05
- link virtual_link2_9: geometry visual box size=0.05 0.002 0.05
- link virtual_link3_1: geometry visual box size=0.025 0.002 0.05
- link virtual_link3_10: geometry visual box size=0.05 0.002 0.05
- link virtual_link3_11: geometry visual box size=0.025 0.002 0.05
- link virtual_link3_2: geometry visual box size=0.05 0.002 0.05
- link virtual_link3_3: geometry visual box size=0.05 0.002 0.05
- link virtual_link3_4: geometry visual box size=0.05 0.002 0.05
- link virtual_link3_5: geometry visual box size=0.05 0.002 0.05
- link virtual_link3_6: geometry visual box size=0.05 0.002 0.05
- link virtual_link3_7: geometry visual box size=0.05 0.002 0.05
- link virtual_link3_8: geometry visual box size=0.05 0.002 0.05
- link virtual_link3_9: geometry visual box size=0.05 0.002 0.05

File: models/three_dof/three_segments/flexible_arm_3dof_3s.urdf (robot description, URDF)
Before this commit: robot flexible_arm, 11 links, 10 joints
Links:
- link virtual_link2_1: geometry visual box size=0.08333333333333333 0.002 0.05
- link virtual_link2_2: geometry visual box size=0.166666667 0.002 0.05
- link virtual_link2_3: geometry visual box size=0.166666667 0.002 0.05
- link virtual_link2_4: geometry visual box size=0.08333333333333333 0.002 0.05
- link virtual_link3_1: geometry visual box size=0.08333333333333333 0.002 0.05
- link virtual_link3_2: geometry visual box size=0.166666667 0.002 0.05
- link virtual_link3_3: geometry visual box size=0.166666667 0.002 0.05
- link virtual_link3_4: geometry visual box size=0.08333333333333333 0.002 0.05

File: models/three_dof/zero_segments/flexible_arm_3dof_0s.urdf (robot description, URDF)
Before this commit: robot flexible_arm, 5 links, 4 joints
Links:
- link virtual_link2_1: geometry visual box size=0.5 0.002 0.05
- link virtual_link3_1: geometry visual box size=0.5 0.002 0.05

Commit message: Implemented new visuzlier that can visualize either trajectoery or a single configuration. It also takes the goal position into account. Changed URDF files, now they have a joint for showing the goal position.

File: models/three_dof/five_segments/flexible_arm_3dof_5s.urdf (robot description, URDF)
Before this commit: robot flexible_arm, 15 links, 14 joints
Links:
- added link goal, mass 0; visual sphere radius=0.025
- link load: geometry visual sphere radius=0.025
- link virtual_link2_1: geometry visual box size=0.05 0.0075 0.05
- link virtual_link2_2: geometry visual box size=0.1 0.0075 0.05
- link virtual_link2_3: geometry visual box size=0.1 0.0075 0.05
- link virtual_link2_4: geometry visual box size=0.1 0.0075 0.05
- link virtual_link2_5: geometry visual box size=0.1 0.0075 0.05
- link virtual_link2_6: geometry visual box size=0.05 0.0075 0.05
- link virtual_link3_1: geometry visual box size=0.05 0.0075 0.05
- link virtual_link3_2: geometry visual box size=0.1 0.0075 0.05
- link virtual_link3_3: geometry visual box size=0.1 0.0075 0.05
- link virtual_link3_4: geometry visual box size=0.1 0.0075 0.05
- link virtual_link3_5: geometry visual box size=0.1 0.0075 0.05
- link virtual_link3_6: geometry visual box size=0.05 0.0075 0.05
Joints:
- added joint goal_link_to_world: type floating, parent world, child goal, origin xyz=0 0 0 rpy=0 0 0

File: models/three_dof/ten_segments/flexible_arm_3dof_10s.urdf (robot description, URDF)
Before this commit: robot flexible_arm, 25 links, 24 joints
Links:
- added link goal, mass 0; visual sphere radius=0.025
- link load: geometry visual sphere radius=0.025
- link virtual_link2_1: geometry visual box size=0.025 0.0075 0.05
- link virtual_link2_10: geometry visual box size=0.05 0.0075 0.05
- link virtual_link2_11: geometry visual box size=0.025 0.0075 0.05
- link virtual_link2_2: geometry visual box size=0.05 0.0075 0.05
- link virtual_link2_3: geometry visual box size=0.05 0.0075 0.05
- link virtual_link2_4: geometry visual box size=0.05 0.0075 0.05
- link virtual_link2_5: geometry visual box size=0.05 0.0075 0.05
- link virtual_link2_6: geometry visual box size=0.05 0.0075 0.05
- link virtual_link2_7: geometry visual box size=0.05 0.0075 0.05
- link virtual_link2_8: geometry visual box size=0.05 0.0075 0.05
- link virtual_link2_9: geometry visual box size=0.05 0.0075 0.05
- link virtual_link3_1: geometry visual box size=0.025 0.0075 0.05
- link virtual_link3_10: geometry visual box size=0.05 0.0075 0.05
- link virtual_link3_11: geometry visual box size=0.025 0.0075 0.05
- link virtual_link3_2: geometry visual box size=0.05 0.0075 0.05
- link virtual_link3_3: geometry visual box size=0.05 0.0075 0.05
- link virtual_link3_4: geometry visual box size=0.05 0.0075 0.05
- link virtual_link3_5: geometry visual box size=0.05 0.0075 0.05
- link virtual_link3_6: geometry visual box size=0.05 0.0075 0.05
- link virtual_link3_7: geometry visual box size=0.05 0.0075 0.05
- link virtual_link3_8: geometry visual box size=0.05 0.0075 0.05
- link virtual_link3_9: geometry visual box size=0.05 0.0075 0.05
Joints:
- added joint goal_link_to_world: type floating, parent world, child goal, origin xyz=0 0 0 rpy=0 0 0

File: models/three_dof/three_segments/flexible_arm_3dof_3s.urdf (robot description, URDF)
Before this commit: robot flexible_arm, 11 links, 10 joints
Links:
- added link goal, mass 0; visual sphere radius=0.025
- link load: geometry visual sphere radius=0.025
- link virtual_link2_1: geometry visual box size=0.08333333333333333 0.0075 0.05
- link virtual_link2_2: geometry visual box size=0.166666667 0.0075 0.05
- link virtual_link2_3: geometry visual box size=0.166666667 0.0075 0.05
- link virtual_link2_4: geometry visual box size=0.08333333333333333 0.0075 0.05
- link virtual_link3_1: geometry visual box size=0.08333333333333333 0.0075 0.05
- link virtual_link3_2: geometry visual box size=0.166666667 0.0075 0.05
- link virtual_link3_3: geometry visual box size=0.166666667 0.0075 0.05
- link virtual_link3_4: geometry visual box size=0.08333333333333333 0.0075 0.05
Joints:
- added joint goal_link_to_world: type floating, parent world, child goal, origin xyz=0 0 0 rpy=0 0 0

File: models/three_dof/two_segments/flexible_arm_3dof_2s.urdf (robot description, URDF)
Before this commit: robot flexible_arm, 9 links, 8 joints
Links:
- added link goal, mass 0; visual sphere radius=0.025
- link load: geometry visual sphere radius=0.025
- link virtual_link2_1: geometry visual box size=0.125 0.0075 0.05
- link virtual_link2_2: geometry visual box size=0.25 0.0075 0.05
- link virtual_link2_3: geometry visual box size=0.125 0.0075 0.05
- link virtual_link3_1: geometry visual box size=0.125 0.0075 0.05
- link virtual_link3_2: geometry visual box size=0.25 0.0075 0.05
- link virtual_link3_3: geometry visual box size=0.125 0.0075 0.05
Joints:
- added joint goal_link_to_world: type floating, parent world, child goal, origin xyz=0 0 0 rpy=0 0 0
- joint last_link_to_load: axis 0 0 1 -> (none)

Commit message: Improved random configuration generation by checking the distance between the elbow position and the wall.

File: models/three_dof/five_segments/flexible_arm_3dof_5s.urdf (robot description, URDF)
Before this commit: robot flexible_arm, 15 links, 14 joints
Links:
- added link wall_link, mass 15; collision box size=0.075 2 1; visual box size=2 0.075 1
Joints:
- added joint world_to_wall: type fixed, parent world, child wall_link, origin xyz=0 -0.15 0

File: models/three_dof/one_segments/flexible_arm_3dof_1s.urdf (robot description, URDF)
Before this commit: robot flexible_arm, 7 links, 6 joints
Links:
- added link wall_link, mass 15; collision box size=0.075 2 1; visual box size=2 0.075 1
Joints:
- added joint world_to_wall: type fixed, parent world, child wall_link, origin xyz=0 -0.15 0

File: models/three_dof/three_segments/flexible_arm_3dof_3s.urdf (robot description, URDF)
Before this commit: robot flexible_arm, 11 links, 10 joints
Links:
- added link wall_link, mass 15; collision box size=0.075 2 1; visual box size=2 0.075 1
Joints:
- added joint world_to_wall: type fixed, parent world, child wall_link, origin xyz=0 -0.15 0

File: models/three_dof/two_segments/flexible_arm_3dof_2s.urdf (robot description, URDF)
Before this commit: robot flexible_arm, 9 links, 8 joints
Links:
- added link wall_link, mass 15; collision box size=0.075 2 1; visual box size=2 0.075 1
Joints:
- added joint world_to_wall: type fixed, parent world, child wall_link, origin xyz=0 -0.15 0
